Commit message: compute the odometry using dynamixel wheel service

File: urdf/robot_x.urdf (robot description, URDF)
Before this commit: robot Robot, 5 links, 4 joints
Joints:
- joint B2W1: origin xyz=0.05 0 -0.06 rpy=0 1.570796 0 -> xyz=0.07 0 -0.06 rpy=0 1.570796 0
- joint B2W2: origin xyz=-0.05 0 -0.06 rpy=0 -1.570796 0 -> xyz=-0.07 0 -0.06 rpy=3.141592 1.570796 0

File: urdf/robot_x.xacro (robot description, xacro)
@@ -21,5 +21,5 @@
 					<cylinder length="0.04" radius="${wheel_radius}"/>
 				</geometry>
-				<origin rpy="0 0 0" xyz="0 0 0.07"/>
+				<origin rpy="0 0 0" xyz="0 0 0.05"/>
 				<material name="black">
 					<color rgba="0 0 0 1"/>
@@ -58,5 +58,5 @@
 			<xacro:wheel_shape/>
 		</link>
-		<link name="wheel_2">
+		<link name="wheel_2">s
 			<xacro:wheel_shape/>
 		</link>
@@ -77,5 +77,5 @@
 			<parent link="base_link"/>
 			<child link="wheel_1"/>
-			<origin xyz="0.05 0 ${-(base_size_z/2 + 0.01)}" rpy="0 ${PI/2} 0"/>
+			<origin xyz="0.07 0 ${-(base_size_z/2 + 0.01)}" rpy="0 ${PI/2} 0"/>
 			<axis xyz="0 0 1"/>
 		</joint>
@@ -83,5 +83,5 @@
 			<parent link="base_link"/>
 			<child link="wheel_2"/>
-			<origin xyz="-0.05 0 ${-(base_size_z/2 + 0.01)}" rpy="0 ${-PI/2} 0"/>
+			<origin xyz="-0.07 0 ${-(base_size_z/2 + 0.01)}" rpy="${PI} ${PI/2} 0"/>
 			<axis xyz="0 0 1"/>
 		</joint>

Commit message: generation velocities

File: urdf/robot_x.urdf (robot description, URDF)
Before this commit: robot Robot, 5 links, 4 joints
Links:
- link base_link: geometry visual box size=0.400 .300 0.086
- link kinect: geometry visual box size=0.1 .2 0.045
- link upper_link: geometry visual box size=.080 0.340 0.065; visual box size=.080 0.340 0.065
- link wheel_1: geometry visual cylinder length=0.04 radius=0.0635
- link wheel_2: geometry visual cylinder length=0.04 radius=0.0635
Joints:
- joint B2U: origin xyz=0 0 0.055 rpy=0 0 -1.570796 -> xyz=0 0 0.08109 rpy=0 0 0
- joint B2W1: origin xyz=0.07 0 -0.06 rpy=0 1.570796 0 -> xyz=0 0.07788 -0.0735 rpy=0 1.570796 1.570796
- joint B2W2: origin xyz=-0.07 0 -0.06 rpy=3.141592 1.570796 0 -> xyz=0 -0.07788 -0.0735 rpy=3.141592 1.570796 1.570796
- joint U2K: origin xyz=0.0866 0 0.05 rpy=0 0 0 -> xyz=0.140 0 0.0325 rpy=0 0 0

File: urdf/robot_x.xacro (robot description, xacro)
@@ -3,17 +3,7 @@
 <!--=======================XACRO DEFINE==============================!-->
 		<xacro:property name="PI" value="3.141592"/>
-		<xacro:property name="wheel_radius" value="0.065"/>
-		<xacro:property name="base_size_z" value="0.1"/>
-		<xacro:macro name="upper_shape" params="yaw x_vec y_vec">
-			<visual>
-				<geometry>
-					<box size="0.05 .3 .1"/>
-				</geometry>
-				<origin rpy="0 0 ${yaw}" xyz="${x_vec} ${y_vec} ${base_size_z/2}"/>
-				<material name="brown">
-					<color rgba="0.5 0.4 0.2 1"/>
-				</material>
-			</visual>
-		</xacro:macro>
+		<xacro:property name="wheel_radius" value="0.0635"/>
+		<xacro:property name="base_size_z" value="0.086"/>
+		<xacro:property name="upper_size_z" value="0.065"/>
 		<xacro:macro name="wheel_shape">
 			<visual>
@@ -21,5 +11,5 @@
 					<cylinder length="0.04" radius="${wheel_radius}"/>
 				</geometry>
-				<origin rpy="0 0 0" xyz="0 0 0.05"/>
+				<origin rpy="0 0 0" xyz="0 0 0.1145"/>
 				<material name="black">
 					<color rgba="0 0 0 1"/>
@@ -31,5 +21,5 @@
 			<visual>
 				<geometry>
-					<box size="0.2 .3 ${base_size_z}"/>
+					<box size="0.400 .300 ${base_size_z}"/>
 				</geometry>
 				<origin rpy="0 0 0" xyz="0 0 0"/>
@@ -40,12 +30,36 @@
 		</link>
 		<link name="upper_link">
-			<xacro:upper_shape yaw = "${0}" x_vec="0.0866" y_vec="0"/>
-			<xacro:upper_shape yaw = "${-PI/3}" x_vec="-0.0433" y_vec="0.075"/>
-			<xacro:upper_shape yaw = "${PI/3}" x_vec="-0.0433" y_vec="-0.075"/>
+			<visual>
+				<geometry>
+					<box size=".080 0.340 ${upper_size_z}"/>
+				</geometry>
+				<origin rpy="0 0 0" xyz=".140 0 ${upper_size_z/2}"/>
+				<material name="brown">
+					<color rgba="0.5 0.4 0.2 1"/>
+				</material>
+			</visual>
+			<visual>
+				<geometry>
+					<box size=".080 0.340 ${upper_size_z}"/>
+				</geometry>
+				<origin rpy="0 0 0" xyz="-0.140 0 ${upper_size_z/2}"/>
+				<material name="brown">
+					<color rgba="0.5 0.4 0.2 1"/>
+				</material>
+			</visual>
+			<visual>
+				<geometry>
+					<box size="0.200 .200 ${upper_size_z}"/>
+				</geometry>
+				<origin rpy="0 0 0" xyz="0 0 ${upper_size_z/2}"/>
+				<material name="brown">
+					<color rgba="0.5 0.4 0.2 1"/>
+				</material>
+			</visual>
 		</link>
 		<link name="kinect">
 			<visual>
 				<geometry>
-					<box size="0.08 .2 ${base_size_z-0.02}"/>
+					<box size="0.1 .2 ${upper_size_z-0.02}"/>
 				</geometry>
 				<origin xyz="0 0 0"/>
@@ -65,5 +79,5 @@
 			<parent link="base_link"/>
 			<child link="upper_link"/>
-			<origin xyz="0 0 ${base_size_z/2+0.005}" rpy="0 0 ${-PI/2}"/>
+			<origin xyz="0 0 ${base_size_z/2+0.03809}" rpy="0 0 0"/>
 			<axis xyz="0 0 1"/>
 			<limit effort="1000.0" lower="${-PI}" upper="${PI}" velocity="0.5"/>
@@ -72,10 +86,10 @@
 			<parent link="upper_link"/>
 			<child link="kinect"/>
-			<origin xyz="0.0866 0 ${base_size_z/2}" rpy="0 0 0"/>
+			<origin xyz="0.140 0 ${upper_size_z/2}" rpy="0 0 0"/>
 		</joint>
 		<joint name="B2W1" type="continuous">
 			<parent link="base_link"/>
 			<child link="wheel_1"/>
-			<origin xyz="0.07 0 ${-(base_size_z/2 + 0.01)}" rpy="0 ${PI/2} 0"/>
+			<origin xyz="0 0.07788 ${-(base_size_z/2 + 0.0305)}" rpy="0 ${PI/2} ${PI/2}"/>
 			<axis xyz="0 0 1"/>
 		</joint>
@@ -83,5 +97,5 @@
 			<parent link="base_link"/>
 			<child link="wheel_2"/>
-			<origin xyz="-0.07 0 ${-(base_size_z/2 + 0.01)}" rpy="${PI} ${PI/2} 0"/>
+			<origin xyz="0 -0.07788 ${-(base_size_z/2 + 0.0305)}" rpy="${PI} ${PI/2} ${PI/2}"/>
 			<axis xyz="0 0 1"/>
 		</joint>
